Commit message: update dexhand files

File: assets/robots/shadow_hand/shadow_hand_left.urdf (robot description, URDF)
Before this commit: robot bimanual_shadowhand_motor, 32 links, 31 joints
Links:
- link lfmetacarpal: geometry visual mesh filename=meshes/visual/lf_metacarpal/lf_metacarpal_E3M5_left.obj scale=0.001 0.001 0.001
- link palm: geometry collision box size=0.018 0.024 0.004; collision box size=0.020 0.024 0.040

File: assets/robots/shadow_hand_new/shadow_hand_left.urdf (robot description, URDF)
Before this commit: robot shadow_right, 32 links, 31 joints
Links:
- removed link manipulator
- added link ee_link
- added link forearm, mass 3.0; collision box size=0.07 0.07 0.07; collision mesh filename=meshes/collision/forearm_E3M5.obj scale=0.001 0.001 0.001
- link ffdistal: mass 0.012 -> 0.12; geometry collision mesh filename=meshes/collision/f_distal_pst.obj scale=0.001 0.001 0.001; visual mesh filename=meshes/visual/f_distal_pst.obj scale=0.001 0.001 0.001
- link ffknuckle: geometry collision mesh filename=meshes/collision/f_knuckle_E3M5.obj; visual mesh filename=meshes/visual/f_knuckle_E3M5.obj scale=0.001 0.001 0.001
- link ffmiddle: geometry collision cylinder length=0.025 radius=0.007; collision sphere radius=0.007
- link ffproximal: geometry collision cylinder length=0.040 radius=0.007; visual mesh filename=meshes/visual/f_proximal_E3M5.obj scale=0.001 0.001 0.001
- link lfdistal: mass 0.012 -> 0.12; geometry collision mesh filename=meshes/visual/f_distal_pst.obj scale=0.001 0.001 0.001; visual mesh filename=meshes/visual/f_distal_pst.obj scale=0.001 0.001 0.001
- link lfknuckle: geometry collision mesh filename=meshes/collision/f_knuckle_E3M5.obj; visual mesh filename=meshes/visual/f_knuckle_E3M5.obj scale=0.001 0.001 0.001
- link lfmetacarpal: geometry collision box size=0.018 0.024 0.040; visual mesh filename=meshes/visual/lf_metacarpal_E3M5_left.obj scale=0.001 0.001 0.001
- link lfmiddle: geometry collision cylinder length=0.025 radius=0.007; collision sphere radius=0.007
- link lfproximal: geometry collision cylinder length=0.040 radius=0.007; visual mesh filename=meshes/visual/f_proximal_E3M5.obj scale=0.001 0.001 0.001
- link mfdistal: mass 0.012 -> 0.12; geometry collision mesh filename=meshes/collision/f_distal_pst.obj scale=0.001 0.001 0.001; visual mesh filename=meshes/visual/f_distal_pst.obj scale=0.001 0.001 0.001
- link mfknuckle: geometry collision mesh filename=meshes/collision/f_knuckle_E3M5.obj; visual mesh filename=meshes/visual/f_knuckle_E3M5.obj scale=0.001 0.001 0.001
- link mfmiddle: geometry collision cylinder length=0.025 radius=0.007; collision sphere radius=0.007
- link mfproximal: geometry collision cylinder length=0.040 radius=0.007; visual mesh filename=meshes/visual/f_proximal_E3M5.obj scale=0.001 0.001 0.001
- link palm: geometry collision box size=0.018 0.024 0.004; collision box size=0.020 0.024 0.032
- link rfdistal: mass 0.012 -> 0.12; geometry collision mesh filename=meshes/collision/f_distal_pst.obj scale=0.001 0.001 0.001; visual mesh filename=meshes/visual/f_distal_pst.obj scale=0.001 0.001 0.001
- link rfknuckle: geometry collision mesh filename=meshes/collision/f_knuckle_E3M5.obj; visual mesh filename=meshes/visual/f_knuckle_E3M5.obj scale=0.001 0.001 0.001
- link rfmiddle: geometry collision cylinder length=0.025 radius=0.007; collision sphere radius=0.007
- link rfproximal: geometry collision cylinder length=0.040 radius=0.007; visual mesh filename=meshes/visual/f_proximal_E3M5.obj scale=0.001 0.001 0.001
- link thdistal: mass 0.016 -> 0.16; geometry collision mesh filename=meshes/visual/th_distal_pst.obj scale=0.001 0.001 0.001; visual mesh filename=meshes/visual/th_distal_pst.obj scale=0.001 0.001 0.001
- link thhub: geometry collision sphere radius=0.010
- link thmiddle: geometry collision mesh filename=meshes/collision/th_middle_E3M5.obj scale=0.001 0.001 0.001; visual mesh filename=meshes/visual/th_middle_E3M5.obj scale=0.001 0.001 0.001
- link thproximal: geometry collision mesh filename=meshes/collision/th_proximal_E3M5.obj scale=0.001 0.001 0.001; visual mesh filename=meshes/visual/th_proximal_E3M5.obj scale=0.001 0.001 0.001
- link wrist: geometry collision box size=0.027 0.018 0.010; collision box size=0.027 0.018 0.010
Joints:
- removed joint thtip
- added joint THtip: type fixed, parent thdistal, child thtip, origin xyz=0 0 0.0275 rpy=0 0 0
- added joint WRJ2: type revolute, parent forearm, child wrist, origin xyz=0 -0.010 0.21301 rpy=0 0 0, axis 0 -1 0, limit lower=-0.523598775598 upper=0.174532925199 effort=10 velocity=2.0
- joint FFJ1: limit lower=0 upper=1.571 effort=2 velocity=2.0 -> lower=0 upper=1.57079632679 effort=2 velocity=2.0
- joint FFJ2: limit lower=0 upper=1.571 effort=2 velocity=2.0 -> lower=0 upper=1.57079632679 effort=2 velocity=2.0
- joint FFJ3: limit lower=0.0 upper=1.571 effort=2 velocity=2.0 -> lower=-0.261799387799 upper=1.57079632679 effort=2 velocity=2.0
- joint FFJ4: limit lower=-0.349000 upper=0.349000 effort=2 velocity=2.0 -> lower=-0.349065850399 upper=0.349065850399 effort=2 velocity=2.0; origin xyz=0.033 0 0.095 rpy=0 0 0 -> xyz=-0.033 0 0.095 rpy=0 0 0
- joint LFJ1: limit lower=0 upper=1.571 effort=2 velocity=2.0 -> lower=0 upper=1.57079632679 effort=2 velocity=2.0
- joint LFJ2: limit lower=0 upper=1.571 effort=2 velocity=2.0 -> lower=0 upper=1.57079632679 effort=2 velocity=2.0
- joint LFJ3: limit lower=0.0 upper=1.571 effort=2 velocity=2.0 -> lower=-0.261799387799 upper=1.57079632679 effort=2 velocity=2.0
- joint LFJ4: axis 0 1 0 -> 0 -1 0; limit lower=-0.349 upper=0.349 effort=2 velocity=2.0 -> lower=-0.349065850399 upper=0.349065850399 effort=2 velocity=2.0; origin xyz=0 0 0.06579 rpy=0 0 0 -> xyz=-0.05397275 0 0.03779463 rpy=0 -0.9599 0
- joint LFJ5: axis 0.573576436 0 0.819152044 -> 1 0 0; limit lower=0 upper=0.785 effort=2 velocity=2.0 -> lower=0 upper=0.785398163397 effort=2 velocity=2.0; origin xyz=-0.033 0 0.02071 rpy=0 0 0 -> xyz=0.033 0 0.02071 rpy=0 0.9599 0
- joint MFJ1: limit lower=0 upper=1.571 effort=2 velocity=2.0 -> lower=0 upper=1.57079632679 effort=2 velocity=2.0
- joint MFJ2: limit lower=0 upper=1.571 effort=2 velocity=2.0 -> lower=0 upper=1.57079632679 effort=2 velocity=2.0
- joint MFJ3: limit lower=0.0 upper=1.571 effort=2 velocity=2.0 -> lower=-0.261799387799 upper=1.57079632679 effort=2 velocity=2.0
- joint MFJ4: limit lower=-0.349 upper=0.349 effort=2 velocity=2.0 -> lower=-0.349065850399 upper=0.349065850399 effort=2 velocity=2.0; origin xyz=0.011 0 0.099 rpy=0 0 0 -> xyz=-0.011 0 0.099 rpy=0 0 0
- joint RFJ1: limit lower=0 upper=1.571 effort=2 velocity=2.0 -> lower=0 upper=1.57079632679 effort=2 velocity=2.0
- joint RFJ2: limit lower=0 upper=1.571 effort=2 velocity=2.0 -> lower=0 upper=1.57079632679 effort=2 velocity=2.0
- joint RFJ3: limit lower=0.0 upper=1.571 effort=2 velocity=2.0 -> lower=-0.261799387799 upper=1.57079632679 effort=2 velocity=2.0
- joint RFJ4: axis 0 1 0 -> 0 -1 0; origin xyz=-0.011 0 0.095 rpy=0 0 0 -> xyz=0.011 0 0.095 rpy=0 0 0
- joint THJ1: axis -1 0 0 -> 1 0 0; limit lower=-1.57079632679 upper=0.0 effort=1.0 velocity=4.0 -> lower=-0.261799387799 upper=1.57079632679 effort=1.0 velocity=4.0
- joint THJ2: axis -1 0 0 -> 1 0 0; limit lower=-0.524 upper=0.524 effort=2.0 velocity=2.0 -> lower=-0.698131700798 upper=0.698131700798 effort=2.0 velocity=2.0
- joint THJ3: axis 0 1 0 -> 0 -1 0; limit lower=-0.209 upper=0.209 effort=2.0 velocity=4.0 -> lower=-0.209439510239 upper=0.209439510239 effort=2.0 velocity=4.0
- joint THJ4: axis 0 1 0 -> 0 -1 0; limit lower=0.0 upper=1.222 effort=3 velocity=4.0 -> lower=0.0 upper=1.2217304764 effort=3 velocity=4.0
- joint THJ5: axis 0 0 -1 -> 0 0 1; limit lower=-1.047 upper=1.047 effort=5.0 velocity=4.0 -> lower=-1.0471975512 upper=1.0471975512 effort=5.0 velocity=4.0; origin xyz=0.034 -0.00858 0.029 rpy=-0.785398163397 0 -1.57079632679 -> xyz=-0.034 -0.00858 0.029 rpy=-0.785398163397 0 1.57079632679
- joint WRJ1: axis (none) -> 1 0 0; limit (none) -> lower=-0.698131700798 upper=0.488692190558 effort=30 velocity=2.0; type fixed -> revolute
- joint ee_fixed_joint: child manipulator -> ee_link; origin xyz=0.0 0.0 0.05 rpy=0.0 0.0 0.0 -> xyz=0.0 0.0 0.00 rpy=0.0 0.0 0.0
- joint world_joint: child wrist -> forearm

File: assets/robots/shadow_hand_new/shadow_hand_left_glb.urdf (robot description, URDF)
Before this commit: robot shadow_right, 32 links, 31 joints
Links:
- removed link manipulator
- added link ee_link
- added link forearm, mass 3.0; collision box size=0.07 0.07 0.07; collision mesh filename=meshes/collision/forearm_E3M5.obj scale=0.001 0.001 0.001
- link ffdistal: mass 0.012 -> 0.12; geometry collision mesh filename=meshes/collision/f_distal_pst.obj scale=0.001 0.001 0.001; visual mesh filename=meshes/visual/f_distal_pst.glb scale=0.001 0.001 0.001
- link ffknuckle: geometry collision mesh filename=meshes/collision/f_knuckle_E3M5.obj; visual mesh filename=meshes/visual/f_knuckle_E3M5.glb scale=0.001 0.001 0.001
- link ffmiddle: geometry collision cylinder length=0.025 radius=0.007; collision sphere radius=0.007
- link ffproximal: geometry collision cylinder length=0.040 radius=0.007; visual mesh filename=meshes/visual/f_proximal_E3M5.glb scale=0.001 0.001 0.001
- link lfdistal: mass 0.012 -> 0.12; geometry collision mesh filename=meshes/collision/f_distal_pst.obj scale=0.001 0.001 0.001; visual mesh filename=meshes/visual/f_distal_pst.glb scale=0.001 0.001 0.001
- link lfknuckle: geometry collision mesh filename=meshes/collision/f_knuckle_E3M5.obj; visual mesh filename=meshes/visual/f_knuckle_E3M5.glb scale=0.001 0.001 0.001
- link lfmetacarpal: geometry collision box size=0.018 0.024 0.040; visual mesh filename=meshes/visual/lf_metacarpal_E3M5_left.glb scale=0.001 0.001 0.001
- link lfmiddle: geometry collision cylinder length=0.025 radius=0.007; collision sphere radius=0.007
- link lfproximal: geometry collision cylinder length=0.040 radius=0.007; visual mesh filename=meshes/visual/f_proximal_E3M5.glb scale=0.001 0.001 0.001
- link mfdistal: mass 0.012 -> 0.12; geometry collision mesh filename=meshes/collision/f_distal_pst.obj scale=0.001 0.001 0.001; visual mesh filename=meshes/visual/f_distal_pst.glb scale=0.001 0.001 0.001
- link mfknuckle: geometry collision mesh filename=meshes/collision/f_knuckle_E3M5.obj; visual mesh filename=meshes/visual/f_knuckle_E3M5.glb scale=0.001 0.001 0.001
- link mfmiddle: geometry collision cylinder length=0.025 radius=0.007; collision sphere radius=0.007
- link mfproximal: geometry collision cylinder length=0.040 radius=0.007; visual mesh filename=meshes/visual/f_proximal_E3M5.glb scale=0.001 0.001 0.001
- link palm: geometry collision box size=0.018 0.024 0.004; collision box size=0.020 0.024 0.032
- link rfdistal: mass 0.012 -> 0.12; geometry collision mesh filename=meshes/collision/f_distal_pst.obj scale=0.001 0.001 0.001; visual mesh filename=meshes/visual/f_distal_pst.glb scale=0.001 0.001 0.001
- link rfknuckle: geometry collision mesh filename=meshes/collision/f_knuckle_E3M5.obj; visual mesh filename=meshes/visual/f_knuckle_E3M5.glb scale=0.001 0.001 0.001
- link rfmiddle: geometry collision cylinder length=0.025 radius=0.007; collision sphere radius=0.007
- link rfproximal: geometry collision cylinder length=0.040 radius=0.007; visual mesh filename=meshes/visual/f_proximal_E3M5.glb scale=0.001 0.001 0.001
- link thdistal: mass 0.016 -> 0.16; geometry collision mesh filename=meshes/visual/th_distal_pst.obj scale=0.001 0.001 0.001; visual mesh filename=meshes/visual/th_distal_pst.glb scale=0.001 0.001 0.001
- link thhub: geometry collision sphere radius=0.010
- link thmiddle: geometry collision mesh filename=meshes/collision/th_middle_E3M5.obj scale=0.001 0.001 0.001; visual mesh filename=meshes/visual/th_middle_E3M5.glb scale=0.001 0.001 0.001
- link thproximal: geometry collision mesh filename=meshes/collision/th_proximal_E3M5.obj scale=0.001 0.001 0.001; visual mesh filename=meshes/visual/th_proximal_E3M5.glb scale=0.001 0.001 0.001
- link wrist: geometry collision box size=0.027 0.018 0.010; collision box size=0.027 0.018 0.010
Joints:
- removed joint thtip
- added joint THtip: type fixed, parent thdistal, child thtip, origin xyz=0 0 0.0275 rpy=0 0 0
- added joint WRJ2: type revolute, parent forearm, child wrist, origin xyz=0 -0.010 0.21301 rpy=0 0 0, axis 0 -1 0, limit lower=-0.523598775598 upper=0.174532925199 effort=10 velocity=2.0
- joint FFJ1: limit lower=0 upper=1.571 effort=2 velocity=2.0 -> lower=0 upper=1.57079632679 effort=2 velocity=2.0
- joint FFJ2: limit lower=0 upper=1.571 effort=2 velocity=2.0 -> lower=0 upper=1.57079632679 effort=2 velocity=2.0
- joint FFJ3: limit lower=0.0 upper=1.571 effort=2 velocity=2.0 -> lower=-0.261799387799 upper=1.57079632679 effort=2 velocity=2.0
- joint FFJ4: limit lower=-0.349000 upper=0.349000 effort=2 velocity=2.0 -> lower=-0.349065850399 upper=0.349065850399 effort=2 velocity=2.0; origin xyz=0.033 0 0.095 rpy=0 0 0 -> xyz=-0.033 0 0.095 rpy=0 0 0
- joint LFJ1: limit lower=0 upper=1.571 effort=2 velocity=2.0 -> lower=0 upper=1.57079632679 effort=2 velocity=2.0
- joint LFJ2: limit lower=0 upper=1.571 effort=2 velocity=2.0 -> lower=0 upper=1.57079632679 effort=2 velocity=2.0
- joint LFJ3: limit lower=0.0 upper=1.571 effort=2 velocity=2.0 -> lower=-0.261799387799 upper=1.57079632679 effort=2 velocity=2.0
- joint LFJ4: axis 0 1 0 -> 0 -1 0; limit lower=-0.349 upper=0.349 effort=2 velocity=2.0 -> lower=-0.349065850399 upper=0.349065850399 effort=2 velocity=2.0; origin xyz=0 0 0.06579 rpy=0 0 0 -> xyz=-0.05397275 0 0.03779463 rpy=0 -0.9599 0
- joint LFJ5: axis 0.573576436 0 0.819152044 -> 1 0 0; limit lower=0 upper=0.785 effort=2 velocity=2.0 -> lower=0 upper=0.785398163397 effort=2 velocity=2.0; origin xyz=-0.033 0 0.02071 rpy=0 0 0 -> xyz=0.033 0 0.02071 rpy=0 0.9599 0
- joint MFJ1: limit lower=0 upper=1.571 effort=2 velocity=2.0 -> lower=0 upper=1.57079632679 effort=2 velocity=2.0
- joint MFJ2: limit lower=0 upper=1.571 effort=2 velocity=2.0 -> lower=0 upper=1.57079632679 effort=2 velocity=2.0
- joint MFJ3: limit lower=0.0 upper=1.571 effort=2 velocity=2.0 -> lower=-0.261799387799 upper=1.57079632679 effort=2 velocity=2.0
- joint MFJ4: limit lower=-0.349 upper=0.349 effort=2 velocity=2.0 -> lower=-0.349065850399 upper=0.349065850399 effort=2 velocity=2.0; origin xyz=0.011 0 0.099 rpy=0 0 0 -> xyz=-0.011 0 0.099 rpy=0 0 0
- joint RFJ1: limit lower=0 upper=1.571 effort=2 velocity=2.0 -> lower=0 upper=1.57079632679 effort=2 velocity=2.0
- joint RFJ2: limit lower=0 upper=1.571 effort=2 velocity=2.0 -> lower=0 upper=1.57079632679 effort=2 velocity=2.0
- joint RFJ3: limit lower=0.0 upper=1.571 effort=2 velocity=2.0 -> lower=-0.261799387799 upper=1.57079632679 effort=2 velocity=2.0
- joint RFJ4: axis 0 1 0 -> 0 -1 0; origin xyz=-0.011 0 0.095 rpy=0 0 0 -> xyz=0.011 0 0.095 rpy=0 0 0
- joint THJ1: axis -1 0 0 -> 1 0 0; limit lower=-1.57079632679 upper=0.0 effort=1.0 velocity=4.0 -> lower=-0.261799387799 upper=1.57079632679 effort=1.0 velocity=4.0
- joint THJ2: axis -1 0 0 -> 1 0 0; limit lower=-0.524 upper=0.524 effort=2.0 velocity=2.0 -> lower=-0.698131700798 upper=0.698131700798 effort=2.0 velocity=2.0
- joint THJ3: axis 0 1 0 -> 0 -1 0; limit lower=-0.209 upper=0.209 effort=2.0 velocity=4.0 -> lower=-0.209439510239 upper=0.209439510239 effort=2.0 velocity=4.0
- joint THJ4: axis 0 1 0 -> 0 -1 0; limit lower=0.0 upper=1.222 effort=3 velocity=4.0 -> lower=0.0 upper=1.2217304764 effort=3 velocity=4.0
- joint THJ5: axis 0 0 -1 -> 0 0 1; limit lower=-1.047 upper=1.047 effort=5.0 velocity=4.0 -> lower=-1.0471975512 upper=1.0471975512 effort=5.0 velocity=4.0; origin xyz=0.034 -0.00858 0.029 rpy=-0.785398163397 0 -1.57079632679 -> xyz=-0.034 -0.00858 0.029 rpy=-0.785398163397 0 1.57079632679
- joint WRJ1: axis (none) -> 1 0 0; limit (none) -> lower=-0.698131700798 upper=0.488692190558 effort=30 velocity=2.0; type fixed -> revolute
- joint ee_fixed_joint: child manipulator -> ee_link; origin xyz=0.0 0.0 0.05 rpy=0.0 0.0 0.0 -> xyz=0.0 0.0 0.00 rpy=0.0 0.0 0.0
- joint world_joint: child wrist -> forearm
