Commit message: latest almost work config

File: assets/urdf/objects/cube_multicolor.urdf (robot description, URDF)
Before this commit: robot object, 1 links, 0 joints
Links:
- link object: mass None -> 0.25

Commit message: fix xml bug

File: assets/urdf/objects/cube_multicolor.urdf (robot description, URDF)
Before this commit: robot object, 1 links, 0 joints
Links:
- link object: mass 0.25 -> 0.01
